File: atmega328p-breakout-game/atmega328p-breakout-game.kicad_pcb (KiCad board)
At the start: 2 copper layers, 77.6 x 52.9 mm, 19 parts, among them J1 Conn_Battery 4.5V, SW1 SW_RESET, SW2 SW_MOVE_RIGHT, SW3 SW_MOVE_LEFT, U1 ATmega328P-P, U2 1088AS

Commit message: a
Parts:
- added Q1: DTC114E, Package_TO_SOT_SMD:SOT-23, B.Cu at (125.9, 79.5)
- added Q2: DTC114E, Package_TO_SOT_SMD:SOT-23, B.Cu at (125.9, 84.0)
- added Q3: DTC114E, Package_TO_SOT_SMD:SOT-23, B.Cu at (121.0, 79.5)
- added Q4: DTC114E, Package_TO_SOT_SMD:SOT-23, B.Cu at (121.0, 84.0)
- added Q5: DTC114E, Package_TO_SOT_SMD:SOT-23, B.Cu at (116.1, 79.1)
- added Q6: DTC114E, Package_TO_SOT_SMD:SOT-23, B.Cu at (116.1, 83.5)
- added Q7: DTC114E, Package_TO_SOT_SMD:SOT-23, B.Cu at (111.2, 79.1)
- added Q8: DTC114E, Package_TO_SOT_SMD:SOT-23, B.Cu at (111.2, 83.5)
- added SW4: SW_DPDT_x2, Button_Switch_THT:SW_Slide_SPDT_Straight_CK_OS102011MS2Q, F.Cu at (177.5, 79.5)
- R10, R11, R4, R5, R6, R7, R8, R9: value 1kΩ -> 220Ω; footprint Resistor_THT:R_Axial_DIN0207_L6.3mm_D2.5mm_P7.62mm_Horizontal -> Resistor_SMD:R_0805_2012Metric_Pad1.20x1.40mm_HandSolder; moved to B.Cu
- U2: value 1088AS -> D15881-M-UR3-0-W; footprint LED_1088:LED_1088 -> LED_1588:LED_1588
- moved R4 39.3 mm to (110.0, 103.1)
- moved R11 32.1 mm to (109.9, 99.0)
- moved R5 32.1 mm to (110.0, 106.0), turned to 180 degrees
- moved R10 30.4 mm to (109.9, 96.0)
- moved U1 30.2 mm to (163.4, 70.3)
- moved R6 29.4 mm to (110.0, 109.0), turned to 180 degrees
- moved R9 29.0 mm to (109.9, 93.1)
- moved R7 26.9 mm to (109.9, 87.2)
- moved R8 20.8 mm to (109.9, 90.2), turned to 180 degrees
- moved U2 19.9 mm to (121.0, 67.5)
- moved SW3 18.3 mm to (124.0, 116.5)
- moved R3 18.0 mm to (123.4, 110.5)
- moved J1 16.7 mm to (178.1, 70.5)
- moved SW1 14.7 mm to (164.0, 116.5)
- moved SW2 14.6 mm to (150.0, 116.5)
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Connections:
- J1 pad 1: VCC -> Net-(J1-Pin_1)
- R10 pad 1: /MATRIX_LED_ROW_7_PIN -> /PORTD5
- R10 pad 2: Net-(U2-R7) -> Net-(U2-C6)
- R11 pad 1: /MATRIX_LED_ROW_8_PIN -> /PORTD6
- R11 pad 2: Net-(U2-R8) -> Net-(U2-C4)
- R4 pad 1: /MATRIX_LED_ROW_1_PIN -> Net-(U2-C2)
- R4 pad 2: Net-(U2-R1) -> /PORTB2
- R5 pad 1: Net-(U2-R2) -> Net-(U2-C3)
- R5 pad 2: /MATRIX_LED_ROW_2_PIN -> /PORTB3
- R6 pad 1: Net-(U2-R3) -> Net-(U2-C5)
- R6 pad 2: /MATRIX_LED_ROW_3_PIN -> /PORTB5
- R7 pad 1: /MATRIX_LED_ROW_4_PIN -> /PORTD0
- R7 pad 2: Net-(U2-R4) -> Net-(U2-C8)
- R8 pad 1: Net-(U2-R5) -> /PORTD1
- R8 pad 2: /MATRIX_LED_ROW_5_PIN -> Net-(U2-C7)
- R9 pad 1: /MATRIX_LED_ROW_6_PIN -> /PORTD3
- R9 pad 2: Net-(U2-R6) -> Net-(U2-C1)
- U1 pad 10: /MATRIX_LED_ROW_8_PIN -> /PORTB7
- U1 pad 11: /MATRIX_LED_COL_6_PIN -> /PORTD5
- U1 pad 12: /MATRIX_LED_COL_7_PIN -> /PORTD6
- U1 pad 13: /MATRIX_LED_COL_8_PIN -> /PORTD7
- U1 pad 14: /MATRIX_LED_ROW_1_PIN -> /PORTB0
- U1 pad 15: /MATRIX_LED_ROW_2_PIN -> /PORTB1
- U1 pad 16: /MATRIX_LED_ROW_3_PIN -> /PORTB2
- U1 pad 17: /MATRIX_LED_ROW_4_PIN -> /PORTB3
- U1 pad 18: /MATRIX_LED_ROW_5_PIN -> /PORTB4
- U1 pad 19: /MATRIX_LED_ROW_6_PIN -> /PORTB5
- U1 pad 2: /MATRIX_LED_COL_1_PIN -> /PORTD0
- U1 pad 3: /MATRIX_LED_COL_2_PIN -> /PORTD1
- U1 pad 4: /MATRIX_LED_COL_3_PIN -> /PORTD2
- U1 pad 5: /MATRIX_LED_COL_4_PIN -> /PORTD3
- U1 pad 6: /MATRIX_LED_COL_5_PIN -> /PORTD4
- U1 pad 9: /MATRIX_LED_ROW_7_PIN -> /PORTB6
- U2 pad 1: /MATRIX_LED_COL_4_PIN -> Net-(Q1-C)
- U2 pad 10: Net-(U2-R4) -> Net-(U2-C4)
- U2 pad 11: Net-(U2-R6) -> Net-(U2-C6)
- U2 pad 12: /MATRIX_LED_COL_5_PIN -> Net-(Q7-C)
- U2 pad 13: Net-(U2-R1) -> Net-(U2-C1)
- U2 pad 14: /MATRIX_LED_COL_7_PIN -> Net-(Q6-C)
- U2 pad 15: Net-(U2-R7) -> Net-(U2-C7)
- U2 pad 16: Net-(U2-R8) -> Net-(U2-C8)
- U2 pad 2: /MATRIX_LED_COL_2_PIN -> Net-(Q2-C)
- U2 pad 3: Net-(U2-R2) -> Net-(U2-C2)
- U2 pad 4: Net-(U2-R3) -> Net-(U2-C3)
- U2 pad 5: /MATRIX_LED_COL_1_PIN -> Net-(Q3-C)
- U2 pad 6: Net-(U2-R5) -> Net-(U2-C5)
- U2 pad 7: /MATRIX_LED_COL_3_PIN -> Net-(Q4-C)
- U2 pad 8: /MATRIX_LED_COL_6_PIN -> Net-(Q5-C)
- U2 pad 9: /MATRIX_LED_COL_8_PIN -> Net-(Q8-C)
Routing:
- net /MOVE_RIGHT_SW: track 143.8 -> 0.00 mm
- net /RESET_SW: track 135.4 -> 0.00 mm
- net /MOVE_LEFT_SW: track 126.1 -> 0.00 mm
- net /MATRIX_LED_ROW_6_PIN: track 120.3 -> 0.00 mm
- net /MATRIX_LED_ROW_5_PIN: track 118.1 -> 0.00 mm
- net /MATRIX_LED_ROW_4_PIN: track 115.4 -> 0.00 mm
- net /MATRIX_LED_ROW_3_PIN: track 113.1 -> 0.00 mm
- net /MATRIX_LED_ROW_2_PIN: track 111.1 -> 0.00 mm
- net /MATRIX_LED_ROW_1_PIN: track 93.5 -> 0.00 mm
- net VCC: track 86.3 -> 0.00 mm
- net /MATRIX_LED_ROW_7_PIN: track 73.9 -> 0.00 mm, vias 1 -> 0
- net Net-(U2-R8): track 70.0 -> 0.00 mm
- net /MATRIX_LED_COL_3_PIN: track 69.8 -> 0.00 mm, vias 2 -> 0
- net /MATRIX_LED_ROW_8_PIN: track 69.3 -> 0.00 mm
- net /MATRIX_LED_COL_1_PIN: track 68.0 -> 0.00 mm
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Other:
- board size 77.6 x 52.9 mm -> 122.1 x 98.4 mm
- board text removed: "+"
- board text removed: "0.1μF"
- board text removed: "1088AS"
- board text removed: "10kΩ"
- board text removed: "10μF"
- board text removed: "1kΩ"
- board text removed: "4.5V"
- board text removed: "ATmega328P"
- board text removed: "Breakout Game v0.1.0.0"
- board text removed: "Move Left"
- board text removed: "Move Right"
- board text removed: "Reset"

Commit message: a
Connections:
- U1 pad 23: /MOVE_LEFT_SW -> unconnected-(U1-PC0-Pad23)
- U1 pad 24: /MOVE_RIGHT_SW -> unconnected-(U1-PC1-Pad24)
- U1 pad 27: unconnected-(U1-PC4-Pad27) -> /MOVE_RIGHT_SW
- U1 pad 28: unconnected-(U1-PC5-Pad28) -> /MOVE_LEFT_SW
Routing:
- net VCC: track 0.00 -> 139.0 mm
- net /MOVE_LEFT_SW: track 0.00 -> 82.7 mm
- net /MOVE_RIGHT_SW: track 0.00 -> 66.7 mm
- net /RESET_SW: track 0.00 -> 62.9 mm
- net Net-(J1-Pin_1): track 0.00 -> 9.58 mm

Commit message: aa
Parts:
- moved SW4 0.32 mm to (177.5, 79.8)
Other:
- board size 122.1 x 98.4 mm -> 70.4 x 62.3 mm
- board text added: "+"
- board text added: "0.1μF"
- board text added: "10kΩ"
- board text added: "10μF"
- board text added: "4.5V"
- board text added: "ATmega328P"
- board text added: "SW_MOVE_LEFT"
- board text added: "SW_MOVE_RIGHT"
- board text added: "SW_RESET"
Changed lines of the file:
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@@
 	(footprint "Button_Switch_THT:SW_Slide_SPDT_Straight_CK_OS102011MS2Q"
 		(layer "F.Cu")
-		(at 177.5 79.5)
+		(at 177.470001 79.816911)
 		(descr "CuK miniature slide switch, OS series, SPDT, https://www.ckswitches.com/media/1428/os.pdf")
 		(tags "switch SPDT")
@@
 	)
 	(gr_rect
-		(start 94.62 48.1)
-		(end 216.73 146.48)
+		(start 117.89 64.37)
+		(end 188.29 126.65)
 		(stroke
 			(width 0.05)
@@
 		(layer "Edge.Cuts")
 	)
+	(gr_text "ATmega328P"
+		(at 162.44 106.63 0)
+		(layer "F.SilkS")
+		(effects
+			(font
+				(size 1 1)
+				(thickness 0.15)
+			)
+			(justify left bottom)
+		)
+	)
+	(gr_text "+"
+		(at 177.35 67.47 0)
+		(layer "F.SilkS")
+		(effects
+			(font
+				(size 1 1)
+				(thickness 0.15)
+			)
+			(justify left bottom)
+		)
+	)
+	(gr_text "4.5V"
+		(at 177.76 75.86 0)
+		(layer "F.SilkS")
+		(effects
+			(font
+				(size 1 1)
+				(thickness 0.15)
+			)
+			(justify left bottom)
+		)
+	)
+	(gr_text "0.1μF"
+		(at 179.43 90.45 90)
+		(layer "F.SilkS")
+		(effects
+			(font
+				(size 1 1)
+				(thickness 0.15)
+			)
+			(justify left bottom)
+		)
+	)
+	(gr_text "10μF"
+		(at 181.14 92.34 0)
+		(layer "F.SilkS")
+		(effects
+			(font
+				(size 1 1)
+				(thickness 0.15)
+			)
+			(justify left bottom)
+		)
+	)
+	(gr_text "10kΩ"
+		(at 125.2 113.46 0)
+		(layer "F.SilkS")
+		(effects
+			(font
+				(size 1 1)
+				(thickness 0.15)
+			)
+			(justify left bottom)
+		)
+	)
+	(gr_text "SW_RESET"
+		(at 164.01 123.79 0)
+		(layer "F.SilkS")
+		(effects
+			(font
+				(size 1 1)
+				(thickness 0.15)
+			)
+			(justify left bottom)
+		)
+	)
+	(gr_text "10kΩ"
+		(at 165.33 113.46 0)
+		(layer "F.SilkS")
+		(effects
+			(font
+				(size 1 1)
+				(thickness 0.15)
+			)
+			(justify left bottom)
+		)
+	)
+	(gr_text "SW_MOVE_RIGHT"
+		(at 147.77 123.79 0)
+		(layer "F.SilkS")
+		(effects
+			(font
+				(size 1 1)
+				(thickness 0.15)
+			)
+			(justify left bottom)
+		)
+	)
+	(gr_text "10kΩ"
+		(at 151.21 113.47 0)
+		(layer "F.SilkS")
+		(effects
+			(font
+				(size 1 1)
+				(thickness 0.15)
+			)
+			(justify left bottom)
+		)
+	)
+	(gr_text "SW_MOVE_LEFT"
+		(at 122.26 123.79 0)
+		(layer "F.SilkS")
+		(effects
+			(font
+				(size 1 1)
+				(thickness 0.15)
+			)
+			(justify left bottom)
+		)
+	)
 	(segment
 		(start 148.399 111.481)
@@
 	)
 	(segment
-		(start 181.5 87.4)
-		(end 182.1 88)
-		(width 0.8)
-		(layer "F.Cu")
-		(net 2)
-	)
-	(segment
 		(start 182.1 107.164156)
 		(end 171.163156 118.101)
@@
 	)
 	(segment
+		(start 182.1 88)
+		(end 181.470001 87.370001)
+		(width 0.8)
+		(layer "F.Cu")
+		(net 2)
+	)
+	(segment
 		(start 171.163156 118.101)
 		(end 163.336844 118.101)
@@
 	)
 	(segment
+		(start 181.470001 87.370001)
+		(end 181.470001 79.816911)
+		(width 0.8)
+		(layer "F.Cu")
+		(net 2)
+	)
+	(segment
 		(start 176.6 89.5)
 		(end 176.5 89.5)
@@
 	)
 	(segment
-		(start 181.5 79.5)
-		(end 181.5 87.4)
-		(width 0.8)
-		(layer "F.Cu")
-		(net 2)
-	)
-	(segment
 		(start 175.42 90.58)
 		(end 171 90.58)
@@
 	)
 	(segment
-		(start 179.5 71.9)
-		(end 179.5 79.5)
+		(start 179.470001 79.816911)
+		(end 179.470001 71.870001)
 		(width 0.8)
 		(layer "F.Cu")
@@
 	)
 	(segment
-		(start 178.1 70.5)
-		(end 179.5 71.9)
+		(start 179.470001 71.870001)
+		(end 178.1 70.5)
 		(width 0.8)
 		(layer "F.Cu")
@@
 		(polygon
 			(pts
-				(xy 109.236784 45.311602) (xy 248.316784 50.601602) (xy 246.256784 155.331602) (xy 75.546784 149.701602)
-				(xy 89.156784 45.811602)
+				(xy 115.77 42.99) (xy 224.88 48.07) (xy 223.843216 137.208398) (xy 82.08 147.38) (xy 95.69 43.49)
 			)
 		)

Commit message: a
Connections:
- Q6 pad 1: /PORTD2 -> /PORTC4
- R9 pad 1: /PORTD3 -> /PORTC5
- U1 pad 27: /MOVE_RIGHT_SW -> /PORTC4
- U1 pad 28: /MOVE_LEFT_SW -> /PORTC5
- U1 pad 4: /PORTD2 -> /MOVE_RIGHT_SW
- U1 pad 5: /PORTD3 -> /MOVE_LEFT_SW
Routing:
- net /MOVE_LEFT_SW: track 82.7 -> 90.0 mm
- net /RESET_SW: track 62.9 -> 61.3 mm
- net /MOVE_RIGHT_SW: track 66.7 -> 68.2 mm
Changed lines of the file:
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@@
 	(net 15 "Net-(Q5-C)")
 	(net 16 "/PORTB7")
-	(net 17 "/PORTD2")
+	(net 17 "/PORTC4")
 	(net 18 "Net-(Q6-C)")
 	(net 19 "Net-(Q7-C)")
@@
 	(net 37 "Net-(U2-C7)")
 	(net 38 "Net-(U2-C1)")
-	(net 39 "/PORTD3")
+	(net 39 "/PORTC5")
 	(net 40 "Net-(U2-C6)")
 	(net 41 "/PORTD5")
@@
 			(layers "*.Cu" "*.Mask")
 			(remove_unused_layers no)
-			(net 17 "/PORTD2")
+			(net 4 "/MOVE_RIGHT_SW")
 			(pinfunction "PD2")
 			(pintype "bidirectional")
@@
 			(layers "*.Cu" "*.Mask")
 			(remove_unused_layers no)
-			(net 39 "/PORTD3")
+			(net 5 "/MOVE_LEFT_SW")
 			(pinfunction "PD3")
 			(pintype "bidirectional")
@@
 			(layers "*.Cu" "*.Mask")
 			(remove_unused_layers no)
-			(net 4 "/MOVE_RIGHT_SW")
+			(net 17 "/PORTC4")
 			(pinfunction "PC4")
 			(pintype "bidirectional")
@@
 			(layers "*.Cu" "*.Mask")
 			(remove_unused_layers no)
-			(net 5 "/MOVE_LEFT_SW")
+			(net 39 "/PORTC5")
 			(pinfunction "PC5")
 			(pintype "bidirectional")
@@
 			(layers "B.Cu" "B.Mask" "B.Paste")
 			(roundrect_rratio 0.25)
-			(net 17 "/PORTD2")
+			(net 17 "/PORTC4")
 			(pinfunction "B")
 			(pintype "input")
@@
 			(layers "B.Cu" "B.Mask" "B.Paste")
 			(roundrect_rratio 0.208333)
-			(net 39 "/PORTD3")
+			(net 39 "/PORTC5")
 			(pintype "passive")
 		)
@@
 	)
 	(segment
-		(start 158 100)
-		(end 158 74.5)
+		(start 166.98 110.5)
+		(end 160.69 104.21)
 		(width 0.3)
 		(layer "F.Cu")
@@
 	)
 	(segment
-		(start 158 74.5)
-		(end 162.24 70.26)
+		(start 171.12 115.88)
+		(end 170.5 116.5)
 		(width 0.3)
 		(layer "F.Cu")
@@
 	)
 	(segment
-		(start 171.12 115.88)
-		(end 170.5 116.5)
+		(start 171.12 110.5)
+		(end 166.98 110.5)
 		(width 0.3)
 		(layer "F.Cu")
@@
 	)
 	(segment
-		(start 162.24 70.26)
-		(end 163.38 70.26)
+		(start 160.69 104.21)
+		(end 160.69 72.25)
 		(width 0.3)
 		(layer "F.Cu")
@@
 	)
 	(segment
-		(start 168.5 110.5)
-		(end 158 100)
+		(start 160.69 72.25)
+		(end 162.68 70.26)
 		(width 0.3)
 		(layer "F.Cu")
@@
 	)
 	(segment
-		(start 171.12 110.5)
-		(end 168.5 110.5)
+		(start 162.68 70.26)
+		(end 163.38 70.26)
 		(width 0.3)
 		(layer "F.Cu")
@@
 	(segment
 		(start 157 110.5)
-		(end 157 74.341565)
+		(end 159.59 107.91)
 		(width 0.3)
 		(layer "F.Cu")
@@
 	)
 	(segment
-		(start 168.088435 72.8)
-		(end 171 72.8)
+		(start 162.341565 69)
+		(end 164.288435 69)
 		(width 0.3)
 		(layer "F.Cu")
@@
 	)
 	(segment
-		(start 157 74.341565)
-		(end 162.341565 69)
+		(start 159.59 107.91)
+		(end 159.59 71.751565)
+		(width 0.3)
+		(layer "F.Cu")
+		(net 4)
+	)
+	(segment
+		(start 164.99 69.701565)
+		(end 164.99 76.27)
 		(width 0.3)
 		(layer "F.Cu")
@@
 	)
 	(segment
-		(start 162.341565 69)
-		(end 164.288435 69)
+		(start 164.288435 69)
+		(end 164.99 69.701565)
 		(width 0.3)
 		(layer "F.Cu")
@@
 	)
 	(segment
-		(start 156.5 116.5)
-		(end 150 116.5)
+		(start 164.99 76.27)
+		(end 163.38 77.88)
 		(width 0.3)
 		(layer "F.Cu")
@@
 	)
 	(segment
-		(start 164.288435 69)
-		(end 168.088435 72.8)
+		(start 159.59 71.751565)
+		(end 162.341565 69)
 		(width 0.3)
 		(layer "F.Cu")
@@
 	)
 	(segment
-		(start 156 93.5)
-		(end 156 74)
+		(start 156.5 116.5)
+		(end 150 116.5)
 		(width 0.3)
 		(layer "F.Cu")
-		(net 5)
+		(net 4)
 	)
 	(segment
-		(start 166.83224 70.26)
-		(end 171 70.26)
+		(start 131 110.5)
+		(end 139 110.5)
 		(width 0.3)
 		(layer "F.Cu")
@@
 	)
 	(segment
-		(start 164.57224 68)
-		(end 166.83224 70.26)
+		(start 158.5 91)
+		(end 158.5 71.5)
 		(width 0.3)
 		(layer "F.Cu")
@@
 	)
 	(segment
-		(start 131 110.5)
-		(end 139 110.5)
+		(start 166.04 78.89137)
+		(end 164.51137 80.42)
 		(width 0.3)
 		(layer "F.Cu")
@@
 	)
 	(segment
-		(start 131 110.5)
-		(end 131 116)
+		(start 161.83 68.17)
+		(end 164.74224 68.17)
 		(width 0.3)
 		(layer "F.Cu")
@@
 	)
 	(segment
-		(start 156 74)
-		(end 162 68)
+		(start 166.04 69.46776)
+		(end 166.04 78.89137)
 		(width 0.3)
 		(layer "F.Cu")
@@
 	)
 	(segment
-		(start 162 68)
-		(end 164.57224 68)
+		(start 164.74224 68.17)
+		(end 166.04 69.46776)
 		(width 0.3)
 		(layer "F.Cu")
@@
 	(segment
 		(start 139 110.5)
-		(end 156 93.5)
+		(end 158.5 91)
+		(width 0.3)
+		(layer "F.Cu")
+		(net 5)
+	)
+	(segment
+		(start 158.5 71.5)
+		(end 161.83 68.17)
+		(width 0.3)
+		(layer "F.Cu")
+		(net 5)
+	)
+	(segment
+		(start 131 110.5)
+		(end 131 116)
+		(width 0.3)
+		(layer "F.Cu")
+		(net 5)
+	)
+	(segment
+		(start 164.51137 80.42)
+		(end 163.38 80.42)
 		(width 0.3)
 		(layer "F.Cu")
@@
 		(min_thickness 0.25)
 		(filled_areas_thickness no)
-		(fill
+		(fill yes
 			(thermal_gap 0.5)
 			(thermal_bridge_width 0.5)

Commit message: a
Parts:
- moved R1 7.65 mm to (171.2, 110.5), turned to 180 degrees
Routing:
- net /RESET_SW: track 61.3 -> 56.5 mm
- net VCC: track 138.7 -> 136.6 mm
- net /MOVE_LEFT_SW: track 90.0 -> 91.1 mm
Other:
- board text added: "Breakout Game v0.1.0.0"
Changed lines of the file:
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@@
 		)
 		(fp_arc
-			(start -0.014214 16.385786)
-			(mid 1.4 16.971572)
-			(end 1.985786 18.385786)
+			(start -0.014214 16.414214)
+			(mid 1.4 17)
+			(end 1.985786 18.414214)
 			(stroke
 				(width 0.12)
@@
 		)
 		(fp_circle
-			(center 1.905 2.03)
-			(end 1.905 0.911966)
+			(center 2.1 35.8)
+			(end 2.1 34.681966)
 			(stroke
 				(width 0.12)
@@
 		)
 		(pad "1" thru_hole circle
-			(at 8.84 30.1)
+			(at 10.01 33)
 			(size 1.7 1.7)
 			(drill 1)
@@
 		)
 		(pad "2" thru_hole circle
-			(at 11.38 30.1)
+			(at 12.55 33)
 			(size 1.7 1.7)
 			(drill 1)
@@
 		)
 		(pad "3" thru_hole circle
-			(at 13.92 30.1)
+			(at 15.09 33)
 			(size 1.7 1.7)
 			(drill 1)
@@
 		)
 		(pad "4" thru_hole circle
-			(at 16.46 30.1)
+			(at 17.63 33)
 			(size 1.7 1.7)
 			(drill 1)
@@
 		)
 		(pad "5" thru_hole circle
-			(at 19 30.1)
+			(at 20.17 33)
 			(size 1.7 1.7)
 			(drill 1)
@@
 		)
 		(pad "6" thru_hole circle
-			(at 21.54 30.1)
+			(at 22.71 33)
 			(size 1.7 1.7)
 			(drill 1)
@@
 		)
 		(pad "7" thru_hole circle
-			(at 24.08 30.1)
+			(at 25.25 33)
 			(size 1.7 1.7)
 			(drill 1)
@@
 		)
 		(pad "8" thru_hole circle
-			(at 26.62 30.1)
+			(at 27.79 33)
 			(size 1.7 1.7)
 			(drill 1)
@@
 		)
 		(pad "9" thru_hole circle
-			(at 29 9.5)
+			(at 27.79 4.8)
 			(size 1.7 1.7)
 			(drill 1)
@@
 		)
 		(pad "10" thru_hole circle
-			(at 26.46 9.5)
+			(at 25.25 4.8)
 			(size 1.7 1.7)
 			(drill 1)
@@
 		)
 		(pad "11" thru_hole circle
-			(at 23.92 9.5)
+			(at 22.71 4.8)
 			(size 1.7 1.7)
 			(drill 1)
@@
 		)
 		(pad "12" thru_hole circle
-			(at 21.38 9.5)
+			(at 20.17 4.8)
 			(size 1.7 1.7)
 			(drill 1)
@@
 		)
 		(pad "13" thru_hole circle
-			(at 18.84 9.5)
+			(at 17.63 4.8)
 			(size 1.7 1.7)
 			(drill 1)
@@
 		)
 		(pad "14" thru_hole circle
-			(at 16.3 9.5)
+			(at 15.09 4.8)
 			(size 1.7 1.7)
 			(drill 1)
@@
 		)
 		(pad "15" thru_hole circle
-			(at 13.76 9.5)
+			(at 12.55 4.8)
 			(size 1.7 1.7)
 			(drill 1)
@@
 		)
 		(pad "16" thru_hole circle
-			(at 11.22 9.5)
+			(at 10.01 4.8)
 			(size 1.7 1.7)
 			(drill 1)
@@
 	(footprint "Resistor_THT:R_Axial_DIN0207_L6.3mm_D2.5mm_P7.62mm_Horizontal"
 		(layer "F.Cu")
-		(at 163.5 110.5)
+		(at 171.15 110.5 180)
 		(descr "Resistor, Axial_DIN0207 series, Axial, Horizontal, pin pitch=7.62mm, 0.25W = 1/4W, length*diameter=6.3*2.5mm^2, http://cdn-reichelt.de/documents/datenblatt/B400/1_4W%23YAG.pdf")
 		(tags "Resistor Axial_DIN0207 series Axial Horizontal pin pitch 7.62mm 0.25W = 1/4W length 6.3mm diameter 2.5mm")
 		(property "Reference" "R1"
-			(at 3.81 -2.37 0)
+			(at 3.8 2.4 0)
 			(layer "F.SilkS")
 			(effects
@@
 		(attr through_hole)
 		(fp_line
-			(start 0.54 -1.37)
-			(end 7.08 -1.37)
+			(start 7.08 1.37)
+			(end 7.08 1.04)
 			(stroke
 				(width 0.12)
@@
 		)
 		(fp_line
-			(start 0.54 -1.04)
-			(end 0.54 -1.37)
+			(start 7.08 -1.37)
+			(end 7.08 -1.04)
 			(stroke
 				(width 0.12)
@@
 		)
 		(fp_line
-			(start 0.54 1.04)
-			(end 0.54 1.37)
+			(start 0.54 1.37)
+			(end 7.08 1.37)
 			(stroke
 				(width 0.12)
@@
 		)
 		(fp_line
-			(start 0.54 1.37)
-			(end 7.08 1.37)
+			(start 0.54 1.04)
+			(end 0.54 1.37)
 			(stroke
 				(width 0.12)
@@
 		)
 		(fp_line
-			(start 7.08 -1.37)
-			(end 7.08 -1.04)
+			(start 0.54 -1.04)
+			(end 0.54 -1.37)
 			(stroke
 				(width 0.12)
@@
 		)
 		(fp_line
-			(start 7.08 1.37)
-			(end 7.08 1.04)
+			(start 0.54 -1.37)
+			(end 7.08 -1.37)
 			(stroke
 				(width 0.12)
@@
 		)
 		(fp_line
-			(start 0 0)
-			(end 0.66 0)
+			(start 7.62 0)
+			(end 6.96 0)
 			(stroke
 				(width 0.1)
@@
 		)
 		(fp_line
-			(start 7.62 0)
-			(end 6.96 0)
+			(start 0 0)
+			(end 0.66 0)
 			(stroke
 				(width 0.1)
@@
 		)
 		(pad "1" thru_hole circle
-			(at 0 0)
+			(at 0 0 180)
 			(size 1.6 1.6)
 			(drill 0.8)
@@
 		)
 		(pad "2" thru_hole circle
-			(at 7.62 0)
+			(at 7.62 0 180)
 			(size 1.6 1.6)
 			(drill 0.8)
@@
 	)
 	(gr_rect
+		(start 173.25 95.5)
+		(end 185.55 123.6)
+		(stroke
+			(width 0.15)
+			(type solid)
+		)
+		(fill no)
+		(layer "F.SilkS")
+	)
+	(gr_rect
 		(start 117.89 64.37)
 		(end 188.29 126.65)
@@
 		)
 	)
+	(gr_text "Breakout Game\nv0.1.0.0"
+		(at 179.35 110.65 0)
+		(layer "F.SilkS")
+		(effects
+			(font
+				(size 1 1)
+				(thickness 0.15)
+			)
+			(justify bottom)
+		)
+	)
 	(gr_text "0.1μF"
 		(at 179.43 90.45 90)
@@
 	)
 	(segment
+		(start 171.15 110.5)
+		(end 171.15 113.7)
+		(width 0.8)
+		(layer "F.Cu")
+		(net 2)
+	)
+	(segment
+		(start 173.357078 115.907078)
+		(end 171.163156 118.101)
+		(width 0.8)
+		(layer "F.Cu")
+		(net 2)
+	)
+	(segment
+		(start 171.15 113.7)
+		(end 173.357078 115.907078)
+		(width 0.8)
+		(layer "F.Cu")
+		(net 2)
+	)
+	(segment
 		(start 149.336844 118.101)
 		(end 148.399 117.163156)
@@
 	)
 	(segment
-		(start 162.399 111.601)
-		(end 163.5 110.5)
-		(width 0.8)
-		(layer "F.Cu")
-		(net 2)
-	)
-	(segment
 		(start 171 90.58)
 		(end 168.46 90.58)
@@
 	(segment
 		(start 182.1 107.164156)
-		(end 171.163156 118.101)
-		(width 0.8)
-		(layer "F.Cu")
-		(net 2)
-	)
-	(segment
-		(start 163.336844 118.101)
-		(end 162.399 117.163156)
+		(end 173.357078 115.907078)
 		(width 0.8)
 		(layer "F.Cu")
@@
 	)
 	(segment
-		(start 162.399 117.163156)
-		(end 162.399 111.601)
-		(width 0.8)
-		(layer "F.Cu")
-		(net 2)
-	)
-	(segment
 		(start 182.1 88)
 		(end 181.470001 87.370001)
@@
 	)
 	(segment
-		(start 166.98 110.5)
-		(end 160.69 104.21)
+		(start 163.53 110.5)
+		(end 163.53 116.03)
 		(width 0.3)
 		(layer "F.Cu")
@@
 	)
 	(segment
-		(start 171.12 110.5)
-		(end 166.98 110.5)
-		(width 0.3)
-		(layer "F.Cu")
-		(net 3)
-	)
-	(segment
 		(start 170.5 116.5)
 		(end 164 116.5)
@@
 	)
 	(segment
-		(start 160.69 104.21)
+		(start 160.69 107.66)
 		(end 160.69 72.25)
 		(width 0.3)
@@
 	)
 	(segment
-		(start 162.68 70.26)
-		(end 163.38 70.26)
+		(start 163.53 110.5)
+		(end 160.69 107.66)
 		(width 0.3)
 		(layer "F.Cu")
@@
 	)
 	(segment
-		(start 171.12 110.5)
-		(end 171.12 115.88)
+		(start 163.53 116.03)
+		(end 164 116.5)
+		(width 0.3)
+		(layer "F.Cu")
+		(net 3)
+	)
+	(segment
+		(start 162.68 70.26)
+		(end 163.38 70.26)
 		(width 0.3)
 		(layer "F.Cu")
@@
 	)
 	(segment
-		(start 131 110.5)
-		(end 139 110.5)
+		(start 130.5 116.5)
+		(end 124 116.5)
 		(width 0.3)
 		(layer "F.Cu")
@@
 	)
 	(segment
-		(start 130.5 116.5)
-		(end 124 116.5)
+		(start 161.83 68.17)
+		(end 164.74224 68.17)
 		(width 0.3)
 		(layer "F.Cu")
@@
 	)
 	(segment
-		(start 158.5 91)
-		(end 158.5 71.5)
+		(start 164.74224 68.17)
+		(end 166.04 69.46776)
 		(width 0.3)
 		(layer "F.Cu")
@@
 	)
 	(segment
-		(start 166.04 78.89137)
-		(end 164.51137 80.42)
+		(start 166.04 69.46776)
+		(end 166.04 78.89137)
 		(width 0.3)
 		(layer "F.Cu")
@@
 	)
 	(segment
-		(start 161.83 68.17)
-		(end 164.74224 68.17)
+		(start 164.51137 80.42)
+		(end 163.38 80.42)
 		(width 0.3)
 		(layer "F.Cu")
@@
 	)
 	(segment
-		(start 166.04 69.46776)
-		(end 166.04 78.89137)
+		(start 131 110.5)
+		(end 141 110.5)
 		(width 0.3)
 		(layer "F.Cu")
@@
 	)
 	(segment
-		(start 164.74224 68.17)
-		(end 166.04 69.46776)
+		(start 158.5 93)
+		(end 158.5 71.5)
 		(width 0.3)
 		(layer "F.Cu")
@@
 	)
 	(segment
-		(start 139 110.5)
-		(end 158.5 91)
+		(start 131 110.5)
+		(end 131 116)
 		(width 0.3)
 		(layer "F.Cu")
@@
 	)
 	(segment
-		(start 131 110.5)
-		(end 131 116)
+		(start 141 110.5)
+		(end 158.5 93)
 		(width 0.3)
 		(layer "F.Cu")
@@
 	)
 	(segment
-		(start 164.51137 80.42)
-		(end 163.38 80.42)
+		(start 166.04 78.89137)
+		(end 164.51137 80.42)
 		(width 0.3)
 		(layer "F.Cu")
@@
 		(min_thickness 0.25)
 		(filled_areas_thickness no)
-		(fill yes
+		(fill
 			(thermal_gap 0.5)
 			(thermal_bridge_width 0.5)
