File: atmega328p-breakout-game/atmega328p-breakout-game.kicad_pcb (KiCad board)
At the start: 2 copper layers, 70.4 x 62.3 mm, 28 parts, among them J1 Conn_Battery 4.5V, Q1 DTC114E, Q2 DTC114E, Q3 DTC114E, Q4 DTC114E, Q5 DTC114E, Q6 DTC114E, Q7 DTC114E, Q8 DTC114E, SW1 SW_RESET, SW2 SW_MOVE_RIGHT, SW3 SW_MOVE_LEFT, SW4 SW_DPDT_x2, U1 ATmega328P-P, U2 D15881-M-UR3-0-W

Commit message: a
Parts:
- moved R11 45.8 mm to (149.6, 76.1)
- moved Q5 45.0 mm to (153.0, 104.9), turned to 90 degrees
- moved Q8 44.0 mm to (152.3, 67.9), turned to -90 degrees
- moved R10 40.6 mm to (145.3, 76.1)
- moved R6 39.7 mm to (147.9, 96.9), turned to 0 degrees
- moved Q7 36.2 mm to (145.6, 67.9), turned to -90 degrees
- moved R9 35.4 mm to (140.9, 76.1)
- moved R5 34.8 mm to (143.6, 97.0), turned to 0 degrees
- moved Q4 32.9 mm to (146.4, 104.9), turned to 90 degrees
- moved Q3 31.7 mm to (140.0, 104.9), turned to 90 degrees
- moved R8 30.0 mm to (136.5, 76.1)
- moved R4 30.0 mm to (139.3, 97.0), turned to 0 degrees
- moved Q6 27.7 mm to (138.9, 67.9), turned to -90 degrees
- moved Q1 25.4 mm to (127.2, 104.9), turned to 90 degrees
- moved R7 24.7 mm to (132.0, 76.1)
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Connections:
- Q1 pad 1: /PORTB0 -> /PORTB5
- Q2 pad 1: /PORTB1 -> /PORTB4
- Q3 pad 1: /PORTB4 -> /PORTB3
- Q4 pad 1: /PORTB6 -> /PORTB2
- Q5 pad 1: /PORTB7 -> /PORTB1
- Q6 pad 1: /PORTC4 -> /PORTC5
- Q7 pad 1: /PORTD4 -> /PORTC4
- Q8 pad 1: /PORTD7 -> /PORTD0
- R10 pad 1: /PORTD5 -> /PORTD4
- R11 pad 1: /PORTD6 -> /PORTD1
- R4 pad 2: /PORTB2 -> /PORTD6
- R5 pad 2: /PORTB3 -> /PORTD7
- R6 pad 2: /PORTB5 -> /PORTB0
- R7 pad 1: /PORTD0 -> /PORTD5
- R8 pad 1: /PORTD1 -> /PORTB7
- R9 pad 1: /PORTC5 -> /PORTB6
Routing:
- net /PORTB5: track 0.00 -> 63.6 mm
- net /PORTB4: track 0.00 -> 53.2 mm
- net /PORTB3: track 0.00 -> 42.5 mm
- net /PORTD5: track 0.00 -> 38.5 mm
- net /PORTC5: track 0.00 -> 36.4 mm
- net /PORTB7: track 0.00 -> 33.0 mm
- net /PORTB2: track 0.00 -> 31.9 mm
- net /PORTC4: track 0.00 -> 30.3 mm
- net /PORTB6: track 0.00 -> 27.4 mm
- net /PORTD6: track 0.00 -> 25.4 mm
- net /PORTD7: track 0.00 -> 21.6 mm
- net /PORTD4: track 0.00 -> 19.9 mm
- net /PORTB1: track 0.00 -> 18.1 mm
- net /PORTB0: track 0.00 -> 17.1 mm
- net /PORTD0: track 0.00 -> 15.4 mm
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Other:
- board size 70.4 x 62.3 mm -> 70.4 x 63.6 mm
- board text added: "220Ω"
- board text added: "DTC114E"

Commit message: a
Parts:
- added C3: 0.1μF, Capacitor_SMD:C_0805_2012Metric_Pad1.18x1.45mm_HandSolder, F.Cu at (158.2, 110.1)
- added C4: 0.1μF, Capacitor_SMD:C_0805_2012Metric_Pad1.18x1.45mm_HandSolder, F.Cu at (132.2, 110.1)
- added R12: 1kΩ, Resistor_SMD:R_0805_2012Metric_Pad1.20x1.40mm_HandSolder, F.Cu at (153.3, 110.1)
- added R13: 1kΩ, Resistor_SMD:R_0805_2012Metric_Pad1.20x1.40mm_HandSolder, F.Cu at (127.3, 110.1)
- C1: footprint Capacitor_THT:C_Disc_D3.0mm_W2.0mm_P2.50mm -> Capacitor_SMD:C_0805_2012Metric_Pad1.18x1.45mm_HandSolder
- R1, R2, R3: footprint Resistor_THT:R_Axial_DIN0207_L6.3mm_D2.5mm_P7.62mm_Horizontal -> Resistor_SMD:R_0805_2012Metric_Pad1.20x1.40mm_HandSolder
- moved R1 3.97 mm to (167.3, 109.5)
- moved SW1 1.71 mm to (164.0, 114.8)
- moved SW2 1.71 mm to (150.0, 114.8)
- moved SW3 1.71 mm to (124.0, 114.8)
- moved C1 1.51 mm to (175.1, 89.5)
- moved C2 1.38 mm to (181.5, 86.8)
- moved R3 1.06 mm to (122.4, 110.1), turned to 90 degrees
- moved R2 1.05 mm to (148.4, 110.1), turned to 90 degrees
Connections:
- SW2 pad 1: /MOVE_RIGHT_SW -> Net-(R12-Pad1)
- SW3 pad 1: /MOVE_LEFT_SW -> Net-(R13-Pad1)
Routing:
- net Net-(R12-Pad1): track 0.00 -> 12.3 mm
- net Net-(R13-Pad1): track 0.00 -> 12.3 mm
- net /MOVE_LEFT_SW: track 98.0 -> 87.0 mm
- net VCC: track 136.6 -> 131.8 mm
- net /MOVE_RIGHT_SW: track 68.2 -> 63.7 mm
- net GND: vias 8 -> 10
Other:
- board size 70.4 x 63.6 mm -> 68 x 60 mm
- board text added: "1kΩ"

Commit message: a
Parts:
- moved R6 2.87 mm to (145.6, 95.1)
- moved R4 2.87 mm to (137.1, 95.1)
- moved R5 2.87 mm to (141.4, 95.1)
- moved Q8 2.65 mm to (154.2, 66.0), turned to 180 degrees
- moved Q7 2.52 mm to (147.2, 66.0), turned to 180 degrees
- moved Q6 2.36 mm to (140.3, 66.0), turned to 180 degrees
- moved R10 1.66 mm to (145.3, 77.8)
- moved R11 1.66 mm to (149.6, 77.8)
- moved R7 1.66 mm to (132.0, 77.8)
- moved R8 1.66 mm to (136.5, 77.8)
- moved R9 1.66 mm to (140.9, 77.8)
- moved Q1 1.39 mm to (127.2, 106.3)
- moved Q2 1.39 mm to (133.4, 106.3)
- moved Q3 1.39 mm to (140.0, 106.3)
- moved Q4 1.39 mm to (146.4, 106.3)
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Routing:
- net /PORTD0: track 15.4 -> 11.4 mm
- net /PORTC4: track 30.3 -> 26.6 mm
- net /PORTC5: track 36.4 -> 32.8 mm
- net Net-(Q8-C): track 4.96 -> 8.11 mm
- net Net-(Q6-C): track 4.61 -> 7.62 mm
- net /PORTB0: track 17.1 -> 20.1 mm
- net /PORTD7: track 21.6 -> 24.2 mm
- net Net-(Q7-C): track 5.81 -> 8.38 mm
- net /PORTD6: track 25.4 -> 27.9 mm
- net Net-(U2-C8): track 3.82 -> 5.48 mm
- net Net-(U2-C7): track 4.61 -> 6.27 mm
- net Net-(U2-C6): track 4.06 -> 5.72 mm
- net Net-(U2-C4): track 4.80 -> 6.46 mm
- net Net-(U2-C1): track 4.36 -> 6.02 mm
- net Net-(Q5-C): track 5.88 -> 7.27 mm
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Other:
- board size 68 x 60 mm -> 68 x 61.2 mm
