File: atmega328p-breakout-game/atmega328p-breakout-game.kicad_pcb (KiCad board)
At the start: 2 copper layers, 68 x 61.2 mm, 32 parts, among them J1 Conn_Battery 4.5V, Q1 DTC114E, Q2 DTC114E, Q3 DTC114E, Q4 DTC114E, Q5 DTC114E, Q6 DTC114E, Q7 DTC114E, Q8 DTC114E, SW1 SW_RESET, SW2 SW_MOVE_RIGHT, SW3 SW_MOVE_LEFT, SW4 SW_DPDT_x2, U1 ATmega328P-P, U2 D15881-M-UR3-0-W

Commit message: a
Parts:
- Q1, Q2, Q3, Q4, Q5, Q6, Q7, Q8: value DTC114E -> DTC113Z
Other:
- board text added: "MUN2213"
- board text removed: "DTC114E"

Commit message: a
Parts:
- C3, C4: value 0.1μF -> 1μF
- R12, R13: value 1kΩ -> 10kΩ
Other:
- board text added: "1μF"
- board text removed: "1kΩ"
Changed lines of the file:
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@@
 			)
 		)
-		(property "Value" "0.1μF"
+		(property "Value" "1μF"
 			(at 0 1.68 90)
 			(layer "F.Fab")
@@
 			)
 		)
-		(property "Value" "0.1μF"
+		(property "Value" "1μF"
 			(at 0 1.68 90)
 			(layer "F.Fab")
@@
 			)
 		)
-		(property "Value" "1kΩ"
+		(property "Value" "10kΩ"
 			(at 0 1.65 90)
 			(layer "F.Fab")
@@
 			)
 		)
-		(property "Value" "1kΩ"
+		(property "Value" "10kΩ"
 			(at 0 1.65 90)
 			(layer "F.Fab")
@@
 		)
 	)
-	(gr_text "1kΩ"
-		(at 155.54 111.6 90)
+	(gr_text "10kΩ"
+		(at 155.55 112.08 90)
 		(layer "F.SilkS")
 		(effects
@@
 		)
 	)
-	(gr_text "0.1μF"
-		(at 134.51 112.42 90)
+	(gr_text "1μF"
+		(at 134.56 111.59 90)
 		(layer "F.SilkS")
 		(effects
@@
 		)
 	)
-	(gr_text "1kΩ"
-		(at 129.51 111.6 90)
+	(gr_text "10kΩ"
+		(at 129.5 112.07 90)
 		(layer "F.SilkS")
 		(effects
@@
 		)
 	)
-	(gr_text "0.1μF"
-		(at 160.56 112.42 90)
+	(gr_text "1μF"
+		(at 160.59 111.8 90)
 		(layer "F.SilkS")
 		(effects

Commit message: a
Parts:
- removed C3, C4: 1μF, Capacitor_SMD:C_0805_2012Metric_Pad1.18x1.45mm_HandSolder
- removed R12, R13: 10kΩ, Resistor_SMD:R_0805_2012Metric_Pad1.20x1.40mm_HandSolder
- moved R1 4.20 mm to (163.4, 108.0), turned to 0 degrees
- moved SW1 3.15 mm to (164.0, 111.6)
- moved SW2 3.15 mm to (150.0, 111.6)
- moved SW3 3.15 mm to (124.0, 111.6)
- moved R2 2.31 mm to (149.4, 108.0), turned to 0 degrees
- moved R3 2.31 mm to (123.4, 108.0), turned to 0 degrees
Connections:
- SW2 pad 1: Net-(R12-Pad1) -> /MOVE_RIGHT_SW
- SW3 pad 1: Net-(R13-Pad1) -> /MOVE_LEFT_SW
Routing:
- net Net-(R12-Pad1): track 12.3 -> 0.00 mm
- net Net-(R13-Pad1): track 12.3 -> 0.00 mm
- net /MOVE_LEFT_SW: track 88.1 -> 96.7 mm
- net /RESET_SW: track 56.7 -> 51.1 mm
- net VCC: track 131.8 -> 126.3 mm
- net /MOVE_RIGHT_SW: track 63.7 -> 67.2 mm
- net GND: vias 10 -> 8
Other:
- board size 68 x 61.2 mm -> 68 x 58.4 mm
- board text removed: "1μF"

Commit message: a
Parts:
- moved R3 12.8 mm to (135.4, 112.3), turned to 90 degrees
- moved R2 6.06 mm to (145.1, 112.2), turned to 90 degrees
- moved R1 5.19 mm to (160.4, 112.2), turned to 90 degrees
Routing:
- net VCC: track 126.3 -> 95.8 mm
- net /RESET_SW: track 51.1 -> 54.6 mm
- net /MOVE_LEFT_SW: track 96.7 -> 93.4 mm
- net /MOVE_RIGHT_SW: track 67.2 -> 68.4 mm

Commit message: a
Parts:
- moved R1 0.15 mm to (160.3, 112.2)
Changed lines of the file:
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@@
 	(footprint "Resistor_SMD:R_0805_2012Metric_Pad1.20x1.40mm_HandSolder"
 		(layer "F.Cu")
-		(at 160.41 112.24 90)
+		(at 160.26 112.23 90)
 		(descr "Resistor SMD 0805 (2012 Metric), square (rectangular) end terminal, IPC-7351 nominal with elongated pad for handsoldering. (Body size source: IPC-SM-782 page 72, https://www.pcb-3d.com/wordpress/wp-content/uploads/ipc-sm-782a_amendment_1_and_2.pdf), generated with kicad-footprint-generator")
 		(tags "resistor handsolder")
@@
 	)
 	(gr_text "10kΩ"
-		(at 162.65 114.24 90)
+		(at 162.5 114.23 90)
 		(layer "F.SilkS")
 		(effects
@@
 	)
 	(segment
-		(start 160.813737 111.643737)
-		(end 160.41 111.24)
+		(start 162.68 70.26)
+		(end 160.69 72.25)
 		(width 0.3)
 		(layer "F.Cu")
@@
 	)
 	(segment
-		(start 162.68 70.26)
-		(end 160.69 72.25)
+		(start 160.69 72.25)
+		(end 160.69 108.313737)
 		(width 0.3)
 		(layer "F.Cu")
@@
 	)
 	(segment
-		(start 160.69 72.25)
-		(end 160.69 108.313737)
+		(start 160.673737 111.643737)
+		(end 160.26 111.23)
 		(width 0.3)
 		(layer "F.Cu")
@@
 	(segment
 		(start 164.02 111.643737)
-		(end 160.813737 111.643737)
+		(end 160.673737 111.643737)
 		(width 0.3)
 		(layer "F.Cu")
